Commit message: update mx_urdf  and delete arm_urdf

File: mx_urdf/urdf/mx_urdf.urdf (robot description, URDF)
Before this commit: robot mx_urdf, 9 links, 8 joints
Links:
- link back_omni_link: mass 0.0046004540764873 -> 0.00460045407648728
- link back_omni_wheel_link: mass 0.0179094868522951 -> 0.0201268954931076
- link base_link: mass 2.6824 -> 2.6444
- link front_omni_wheel_link: mass 0.0179094868522951 -> 0.0201268954931076
Joints:
- joint back_omni: origin xyz=-0.109 0 -0.034 rpy=5.91402563680444E-39 6.27500455221378E-39 -1.63202197874526 -> xyz=-0.109 0 -0.034 rpy=-9.96547374531681E-40 8.56494452366143E-39 -2.50364478445485
- joint back_omni_wheel: origin xyz=0 -0.017 -0.0345 rpy=0 1.44757770682335 1.5707963267949 -> xyz=0.0125679822835678 -0.0114475246809032 -0.0344999999999994 rpy=3.14159265358979 -0.820094510728467 -0.738776383504164
- joint camera: origin xyz=-0.105000000000172 0.00100000000031952 0.476 rpy=5.90138314899544E-39 -6.28689575958092E-39 -1.53144402893157E-12 -> xyz=-0.105000000000172 0.00100000000031975 0.376 rpy=5.90138314899544E-39 -6.28689575958092E-39 -1.53144402893157E-12
- joint front_omni: origin xyz=0.109 0 -0.034 rpy=-6.59336456706476E-39 -5.55688087409284E-39 1.62427663724601 -> xyz=0.109000000000001 0 -0.034 rpy=-5.0560979501588E-39 -6.98478738985546E-39 1.38034790661819
- joint front_omni_wheel: axis 0 -1 0 -> 0 1 0; origin xyz=-0.0114883310248948 -0.0125306923297341 -0.0344999999999982 rpy=0 -1.4482024478998 0.828768272940467 -> xyz=0.0144715368252966 -0.00892046085771814 -0.0344999999999997 rpy=0 -1.34064070369349 2.58919123082909
- joint left_wheel: origin xyz=0 0.145 -0.024 rpy=2.74979624140029 5.90138314899544E-39 -1.57079632679643 -> xyz=0 0.132 -0.024 rpy=2.74979624140029 5.90138314899544E-39 -1.57079632679643
- joint right_wheel: origin xyz=0 -0.145 -0.024 rpy=1.5707963267949 -5.90138314899544E-39 1.57079632679337 -> xyz=0 -0.132 -0.024 rpy=1.5707963267949 -5.90138314899544E-39 1.57079632679337
